File: pcb-lt3032.brd (EAGLE design)
At the start: 26.7 x 10.2 mm, 8 parts

Commit message: Add LT3032 Board
Parts:
- added PCB1: LT3032 rev.A, module-footprints:F-LOGO
- C1, C2, C5, C6: value 10u -> 10U
- C3, C4: value 10n -> 10N
Changed lines of the file:
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@@
 <setting verticaltext="up"/>
 </settings>
-<grid distance="0.5" unitdist="mm" unit="mm" style="dots" multiple="1" display="yes" altdistance="0.125" altunitdist="mm" altunit="mm"/>
+<grid distance="0.5" unitdist="mm" unit="mm" style="dots" multiple="1" display="yes" altdistance="0.1" altunitdist="mm" altunit="mm"/>
 <layers>
 <layer number="1" name="Top" color="4" fill="1" visible="no" active="yes"/>
@@
 </element>
 <element name="U1" library="module-footprints" package="F-DIP8-HEATSINK-NOSILK" value="" x="13.5" y="5.5" locked="yes" rot="R270"/>
-<element name="C1" library="capacitors" package="C-1206" value="10u" x="7.25" y="9.25" smashed="yes" rot="MR0">
+<element name="C1" library="capacitors" package="C-1206" value="10U" x="7.25" y="9.25" smashed="yes" rot="MR0">
 <attribute name="NAME" x="3.75" y="9.25" size="0.8128" layer="26" ratio="15" rot="MR90" align="bottom-center"/>
 </element>
-<element name="C2" library="capacitors" package="C-1206" value="10u" x="7.25" y="1.75" smashed="yes" rot="MR180">
+<element name="C2" library="capacitors" package="C-1206" value="10U" x="7.25" y="1.75" smashed="yes" rot="MR180">
 <attribute name="NAME" x="3.75" y="1.75" size="0.8128" layer="26" ratio="15" rot="MR90" align="bottom-center"/>
 </element>
-<element name="C6" library="capacitors" package="C-1206" value="10u" x="12.75" y="1.75" smashed="yes" rot="MR0">
+<element name="C6" library="capacitors" package="C-1206" value="10U" x="12.75" y="1.75" smashed="yes" rot="MR0">
 <attribute name="NAME" x="16.25" y="1.75" size="0.8128" layer="26" ratio="15" rot="MR270" align="bottom-center"/>
 </element>
-<element name="C5" library="capacitors" package="C-1206" value="10u" x="12.75" y="9.25" smashed="yes" rot="MR180">
+<element name="C5" library="capacitors" package="C-1206" value="10U" x="12.75" y="9.25" smashed="yes" rot="MR180">
 <attribute name="NAME" x="16.25" y="9.25" size="0.8128" layer="26" ratio="15" rot="MR270" align="bottom-center"/>
 </element>
-<element name="C3" library="capacitors" package="C-0805" value="10n" x="14" y="5.5" smashed="yes" rot="MR90">
+<element name="C3" library="capacitors" package="C-0805" value="10N" x="14" y="5.5" smashed="yes" rot="MR90">
 <attribute name="NAME" x="15.27" y="5.5" size="0.8128" layer="26" ratio="15" rot="MR90" align="center"/>
 </element>
-<element name="C4" library="capacitors" package="C-0805" value="10n" x="6" y="5.5" smashed="yes" rot="MR270">
+<element name="C4" library="capacitors" package="C-0805" value="10N" x="6" y="5.5" smashed="yes" rot="MR270">
 <attribute name="NAME" x="4.73" y="5.5" size="0.8128" layer="26" ratio="15" rot="MR270" align="center"/>
 </element>
+<element name="PCB1" library="module-footprints" package="F-LOGO" value="LT3032 rev.A" x="22" y="5.5" rot="R90"/>
 </elements>
 <signals>
