File: pcb-lt3032.sch (EAGLE design)
At the start: 8 parts

Commit message: Add LT3032 Board
Parts:
- added PCB1: LT3032 rev.A, module-footprints:GENERIC-LOGO
- C1, C2, C5, C6: value 10u -> 10U; device capacitors:C-1206 -> capacitors:10U
- C3, C4: value 10n -> 10N; device capacitors:C-0805 -> capacitors:10N
Changed lines of the file:
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@@
 <part name="DA1" library="regulators-linear" deviceset="LT3032" device="-12"/>
 <part name="U1" library="module-footprints" deviceset="F-DUAL-SUPPLY" device="-BOARD"/>
-<part name="C1" library="capacitors" deviceset="C" device="-1206" value="10u"/>
-<part name="C2" library="capacitors" deviceset="C" device="-1206" value="10u"/>
-<part name="C6" library="capacitors" deviceset="C" device="-1206" value="10u"/>
-<part name="C5" library="capacitors" deviceset="C" device="-1206" value="10u"/>
-<part name="C3" library="capacitors" deviceset="C" device="-0805" value="10n"/>
-<part name="C4" library="capacitors" deviceset="C" device="-0805" value="10n"/>
+<part name="C1" library="capacitors" deviceset="?" device="10U" value="10U"/>
+<part name="C2" library="capacitors" deviceset="?" device="10U" value="10U"/>
+<part name="C6" library="capacitors" deviceset="?" device="10U" value="10U"/>
+<part name="C5" library="capacitors" deviceset="?" device="10U" value="10U"/>
+<part name="C3" library="capacitors" deviceset="?" device="10N" value="10N"/>
+<part name="C4" library="capacitors" deviceset="?" device="10N" value="10N"/>
 <part name="GND1" library="supply" deviceset="GND" device=""/>
 <part name="GND2" library="supply" deviceset="GND" device=""/>
+<part name="PCB1" library="module-footprints" deviceset="GENERIC" device="-LOGO" value="LT3032 rev.A"/>
 </parts>
 <sheets>
@@
 <instance part="GND1" gate="VR1" x="-43.18" y="-35.56"/>
 <instance part="GND2" gate="VR1" x="48.26" y="-35.56"/>
+<instance part="PCB1" gate="G$1" x="-20.32" y="5.08"/>
 </instances>
 <busses>
