File: pcb-meter.sch (EAGLE design)
At the start: 41 parts

Commit message: Update
Parts:
- added C3, C5, C8, C9: 100n, capacitors:C-050-024X44
- added C4, C6: 10u/35V, capacitors-electrolytic:C-E2-5
- added HL13: BLUE(3MM), optoelectronics:BLUE(3MM)
- added R20: 1.5k, resistors:R-0207/10
Connections:
- new net N$36: DA1.2.IN-, DA1.2.OUT
- net +15V: now also C3.2, C4.+, C5.2, C8.2, C9.2, DA1*.V+, DA2*.V+, DA3*.V+, DA4*.V+
- net -15V: now also C3.1, C5.1, C6.-, C8.1, C9.1, DA1*.V-, DA2*.V-, DA3*.V-, DA4*.V-
- net GND: now also C4.-, C6.+, DA1.2.IN+, HL13.C
- net N$1: now also R20.2
- net N$11: now also DA4.1.IN-; no longer DA4.4.IN-
- net N$12: now also DA4.2.IN-; no longer DA4.3.IN-
- net N$13: now also DA4.4.IN-; no longer DA4.2.IN-
- net N$14: now also DA4.1.OUT; no longer DA4.4.OUT
- net N$15: now also DA4.2.OUT; no longer DA4.3.OUT
- net N$16: now also DA4.4.OUT; no longer DA4.2.OUT
- net N$17: now also DA4.3.OUT; no longer DA4.1.OUT
- net N$18: now also DA3.1.OUT; no longer DA3.4.OUT
- net N$19: now also DA3.2.OUT; no longer DA3.3.OUT
- net N$2: now also R1.1
- net N$20: now also DA3.4.OUT; no longer DA3.2.OUT
- net N$21: now also DA3.3.OUT; no longer DA3.1.OUT
- net N$22: now also DA2.1.OUT; no longer DA2.4.OUT
- net N$23: now also DA2.2.OUT; no longer DA2.3.OUT
- net N$24: now also DA2.4.OUT; no longer DA2.2.OUT
- net N$25: now also DA2.3.OUT; no longer DA2.1.OUT
- net N$26: now also C1.+, R3.2
- net N$27: now also DA4.3.IN-; no longer DA4.1.IN-
- net N$28: now also DA3.1.IN-; no longer DA3.4.IN-
- net N$29: now also DA3.2.IN-; no longer DA3.3.IN-
- net N$30: now also DA3.4.IN-; no longer DA3.2.IN-
- net N$31: now also DA3.3.IN-; no longer DA3.1.IN-
- net N$32: now also DA2.1.IN-; no longer DA2.4.IN-
- net N$33: now also DA2.2.IN-; no longer DA2.3.IN-
- net N$34: now also DA2.4.IN-; no longer DA2.2.IN-
- net N$35: now also DA2.3.IN-; no longer DA2.1.IN-
- net N$9: now also HL13.A, R20.1; no longer C1.+, R3.2
Other:
- moved on the sheet: C1, DA1.1, DA2*, DA2.1, DA2.2, DA2.3, DA2.4, DA3*, DA3.1, DA3.2, DA3.3, DA3.4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

Commit message: Renumber pcb-meter
Parts:
- removed C9: 100n, capacitors:C-050-024X44
- added C7: 1u/50V, capacitors-electrolytic:C-E1,5-4
- C1: value 1u/50V -> 10u/35V; device capacitors-electrolytic:C-E1,5-4 -> capacitors-electrolytic:C-E2-5
- C2: value 47n -> 10u/35V; device capacitors:C-050-025X075 -> capacitors-electrolytic:C-E2-5
- C4, C6: value 10u/35V -> 100n; device capacitors-electrolytic:C-E2-5 -> capacitors:C-050-024X44
- C8: value 100n -> 47n; device capacitors:C-050-024X44 -> capacitors:C-050-025X075
- HL1: value GREEN(3MM) -> BLUE(3MM); device optoelectronics:GREEN(3MM) -> optoelectronics:BLUE(3MM)
- HL12: value RED(3MM) -> YELLOW(3MM); device optoelectronics:RED(3MM) -> optoelectronics:YELLOW(3MM)
- HL13: value BLUE(3MM) -> RED(3MM); device optoelectronics:BLUE(3MM) -> optoelectronics:RED(3MM)
- HL9: value YELLOW(3MM) -> GREEN(3MM); device optoelectronics:YELLOW(3MM) -> optoelectronics:GREEN(3MM)
- R1: value 56k -> 1.5k
- R10: value 2.2k -> 560R
- R11: value 1.5k -> 820R
- R13: value 820R -> 1.5k
- R14: value 560R -> 2.2k
- R15: value 330R -> 3.3k
- R16: value 330R -> 12k
- R17: value 220R -> 5.6k
- R18: value 220R -> 15k
- R19: value 270R -> 1k
- R2: value 150k -> 56k
- R20: value 1.5k -> 180R
- R3: value 1.8k -> 150k
- R4: value 15k -> 1.8k
- R5: value 180R -> 270R
- R6: value 1k -> 220R
- R7: value 12k -> 220R
- R8: value 5.6k -> 330R
- R9: value 3.3k -> 330R
Connections:
- net +15V: now also C1.+, C4.2, C6.2, R17.1, R19.2, R20.2; no longer C2.2, C4.+, C9.2, R5.2, R6.2, R8.1
- net -15V: now also C2.-, C4.1, C6.1, HL13.C, R18.1; no longer C6.-, C8.1, C9.1, HL12.C, R4.1
- net GND: now also C2.+, C7.-, HL1.C, R5.2; no longer C4.-, C6.+, HL13.C, R19.2
- net N$1: now also R1.2; no longer R20.2
- net N$10: now also C8.1, R20.1; no longer C2.1, R5.1
- net N$11: now also DA2.1.IN-, R16.1, R17.2; no longer DA4.1.IN-, R7.1, R8.2
- net N$12: now also DA2.2.IN-, R15.1, R16.2; no longer DA4.2.IN-, R7.2, R9.1
- net N$13: now also DA2.4.IN-, R14.1, R15.2; no longer DA4.4.IN-, R10.1, R9.2
- net N$14: now also DA2.1.OUT, HL12.C, HL13.A; no longer DA4.1.OUT, HL11.C, HL12.A
- net N$15: now also DA2.2.OUT, HL11.C, HL12.A; no longer DA4.2.OUT, HL10.C, HL11.A
- net N$16: now also DA2.4.OUT, HL10.C, HL11.A; no longer DA4.4.OUT, HL10.A, HL9.C
- net N$17: now also DA2.3.OUT, HL10.A, HL9.C; no longer DA4.3.OUT, HL8.C, HL9.A
- net N$18: now also DA4.1.OUT, HL8.C, HL9.A; no longer DA3.1.OUT, HL7.C, HL8.A
- net N$19: now also DA4.2.OUT, HL7.C, HL8.A; no longer DA3.2.OUT, HL6.C, HL7.A
- net N$2: now also R2.1; no longer R1.1
- net N$20: now also DA4.4.OUT, HL6.C, HL7.A; no longer DA3.4.OUT, HL5.C, HL6.A
- net N$21: now also DA4.3.OUT, HL5.C, HL6.A; no longer DA3.3.OUT, HL4.C, HL5.A
- net N$22: now also DA3.1.OUT, HL4.C, HL5.A; no longer DA2.1.OUT, HL3.C, HL4.A
- net N$23: now also DA3.2.OUT, HL3.C, HL4.A; no longer DA2.2.OUT, HL2.C, HL3.A
- net N$24: now also DA3.4.OUT, HL2.C, HL3.A; no longer DA2.4.OUT, HL1.C, HL2.A
- net N$25: now also DA3.3.OUT, HL2.A; no longer DA2.3.OUT, HL1.A
- net N$26: now also C7.+, R4.2; no longer C1.+, R3.2
- net N$27: now also DA2.3.IN-, R13.1, R14.2; no longer DA4.3.IN-, R10.2, R11.1
- net N$28: now also DA4.1.IN-, R13.2; no longer DA3.1.IN-, R11.2
- net N$29: now also DA4.2.IN-, R11.1; no longer DA3.2.IN-, R13.1
- net N$30: now also DA4.4.IN-, R10.1, R11.2; no longer DA3.4.IN-, R13.2, R14.1
- net N$31: now also DA4.3.IN-, R10.2, R9.1; no longer DA3.3.IN-, R14.2, R15.1
- net N$32: now also DA3.1.IN-, R8.1, R9.2; no longer DA2.1.IN-, R15.2, R16.1
- net N$33: now also DA3.2.IN-, R7.1, R8.2; no longer DA2.2.IN-, R16.2, R17.1
- net N$34: now also DA3.4.IN-, R6.1, R7.2; no longer DA2.4.IN-, R17.2, R18.1
- net N$35: now also DA3.3.IN-, R5.1, R6.2; no longer DA2.3.IN-, R18.2, R19.1
- net N$5: now also R2.2, R3.1; no longer R1.2, R2.1
- net N$6: now also R18.2, R19.1; no longer R4.2, R6.1
- net N$8: now also R3.2, R4.1; no longer R2.2, R3.1
- net N$9: now also HL1.A, R1.1; no longer HL13.A, R20.1
Other:
- moved on the sheet: C1, C3, C8, DA2*, DA2.1, DA2.2, DA2.3, DA2.4, DA3*, DA3.1, DA3.2, DA3.3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

Commit message: Remove PP indicator
Parts:
- removed HL1: BLUE(3MM), optoelectronics:BLUE(3MM)
- removed R1: 1.5k, resistors:R-0207/10
Connections:
- removed net N$1: R1.2, XP1.5
- removed net N$9: HL1.A, R1.1
- net GND: no longer HL1.C
Changed lines of the file:
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@@
 <part name="PWR5" library="supply" deviceset="+15V" device=""/>
 <part name="GND5" library="supply" deviceset="GND" device=""/>
-<part name="R1" library="resistors" deviceset="R" device="-0207/10" value="1.5k"/>
-<part name="HL1" library="optoelectronics" deviceset="?(3MM)" device="BLUE"/>
-<part name="GND3" library="supply" deviceset="GND" device=""/>
 <part name="C6" library="capacitors" deviceset="C" device="-050-024X44" value="100n"/>
 <part name="C5" library="capacitors" deviceset="C" device="-050-024X44" value="100n"/>
@@
 <instance part="GND5" gate="VR1" x="96.52" y="12.7"/>
 <instance part="DA1" gate="*" x="71.12" y="96.52"/>
-<instance part="R1" gate="G$1" x="78.74" y="38.1" rot="R90"/>
-<instance part="HL1" gate="G$1" x="78.74" y="27.94" rot="R270"/>
-<instance part="GND3" gate="VR1" x="78.74" y="20.32"/>
 <instance part="C6" gate="G$1" x="60.96" y="96.52" rot="R90"/>
 <instance part="C5" gate="G$1" x="53.34" y="96.52" rot="R90"/>
@@
 </segment>
 <segment>
-<pinref part="HL1" gate="G$1" pin="C"/>
-<pinref part="GND3" gate="VR1" pin="GND"/>
-<wire x1="78.74" y1="25.4" x2="78.74" y2="22.86" width="0.1524" layer="91"/>
-</segment>
-<segment>
 <pinref part="GND1" gate="VR1" pin="GND"/>
 <wire x1="22.86" y1="93.98" x2="22.86" y2="96.52" width="0.1524" layer="91"/>
@@
 <wire x1="30.48" y1="93.98" x2="30.48" y2="96.52" width="0.1524" layer="91"/>
 <junction x="30.48" y="96.52"/>
-</segment>
-</net>
-<net name="N$1" class="0">
-<segment>
-<pinref part="XP1" gate="G$1" pin="5"/>
-<wire x1="71.12" y1="45.72" x2="78.74" y2="45.72" width="0.1524" layer="91"/>
-<pinref part="R1" gate="G$1" pin="2"/>
-<wire x1="78.74" y1="45.72" x2="78.74" y2="43.18" width="0.1524" layer="91"/>
 </segment>
 </net>
@@
 </segment>
 </net>
-<net name="N$9" class="0">
-<segment>
-<pinref part="R1" gate="G$1" pin="1"/>
-<pinref part="HL1" gate="G$1" pin="A"/>
-<wire x1="78.74" y1="33.02" x2="78.74" y2="30.48" width="0.1524" layer="91"/>
-</segment>
-</net>

Commit message: Add Meter Board
Parts:
- added PCB1: R-PREAMP MTR rev.A, module-footprints:GENERIC-LOGO
- C1, C2: value 10u/35V -> 10U/35V; device capacitors-electrolytic:C-E2-5 -> capacitors-electrolytic:10U/35V
- C3, C4, C5, C6: value 100n -> 100N(TH); device capacitors:C-050-024X44 -> capacitors:100N(TH)
- C7: value 1u/50V -> 1U/50V; device capacitors-electrolytic:C-E1,5-4 -> capacitors-electrolytic:1U/50V
- C8: value 47n -> 47N(FILM); device capacitors:C-050-025X075 -> capacitors:47N(FILM)
- R10: value 560R -> 560R(TH); device resistors:R-0207/10 -> resistors:560R(TH)
- R11: value 820R -> 820R(TH); device resistors:R-0207/10 -> resistors:820R(TH)
- R12: value 1.2k -> 1K2(TH); device resistors:R-0207/10 -> resistors:1K2(TH)
- R13: value 1.5k -> 1K5(TH); device resistors:R-0207/10 -> resistors:1K5(TH)
- R14: value 2.2k -> 2K2(TH); device resistors:R-0207/10 -> resistors:2K2(TH)
- R15: value 3.3k -> 3K3(TH); device resistors:R-0207/10 -> resistors:3K3(TH)
- R16: value 12k -> 12K(TH); device resistors:R-0207/10 -> resistors:12K(TH)
- R17: value 5.6k -> 5K6(TH); device resistors:R-0207/10 -> resistors:5K6(TH)
- R18: value 15k -> 15K(TH); device resistors:R-0207/10 -> resistors:15K(TH)
- R19: value 1k -> 1K(TH); device resistors:R-0207/10 -> resistors:1K(TH)
- R2: value 56k -> 56K(TH); device resistors:R-0207/10 -> resistors:56K(TH)
- R20: value 180R -> 180R(TH); device resistors:R-0207/10 -> resistors:180R(TH)
- R3: value 150k -> 150K(TH); device resistors:R-0207/10 -> resistors:150K(TH)
- R4: value 1.8k -> 1K8(TH); device resistors:R-0207/10 -> resistors:1K8(TH)
- R5: value 270R -> 270R(TH); device resistors:R-0207/10 -> resistors:270R(TH)
- R6, R7: value 220R -> 220R(TH); device resistors:R-0207/10 -> resistors:220R(TH)
- R8, R9: value 330R -> 330R(TH); device resistors:R-0207/10 -> resistors:330R(TH)
Changed lines of the file:
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@@
 <layer number="54" name="bGND_GNDA" color="1" fill="9" visible="no" active="no"/>
 <layer number="56" name="wert" color="7" fill="1" visible="no" active="no"/>
+<layer number="57" name="tCAD" color="7" fill="1" visible="no" active="no"/>
 <layer number="90" name="Modules" color="5" fill="1" visible="yes" active="yes"/>
 <layer number="91" name="Nets" color="2" fill="1" visible="yes" active="yes"/>
@@
 <layer number="97" name="Info" color="7" fill="1" visible="yes" active="yes"/>
 <layer number="98" name="Guide" color="6" fill="1" visible="yes" active="yes"/>
+<layer number="99" name="SpiceOrder" color="7" fill="1" visible="no" active="no"/>
 <layer number="100" name="Muster" color="7" fill="1" visible="no" active="no"/>
 <layer number="101" name="Patch_Top" color="12" fill="4" visible="no" active="yes"/>
@@
 <layer number="111" name="LPC17xx" color="7" fill="1" visible="yes" active="yes"/>
 <layer number="112" name="tSilk" color="7" fill="1" visible="yes" active="yes"/>
+<layer number="113" name="ReferenceLS" color="7" fill="1" visible="no" active="no"/>
 <layer number="116" name="Patch_BOT" color="9" fill="4" visible="no" active="yes"/>
+<layer number="118" name="Rect_Pads" color="7" fill="1" visible="no" active="no"/>
 <layer number="121" name="_tsilk" color="7" fill="1" visible="no" active="yes"/>
 <layer number="122" name="_bsilk" color="7" fill="1" visible="no" active="yes"/>
@@
 <layer number="132" name="bAdjust" color="7" fill="1" visible="no" active="yes"/>
 <layer number="144" name="Drill_legend" color="7" fill="1" visible="no" active="yes"/>
+<layer number="150" name="Notes" color="7" fill="1" visible="no" active="yes"/>
 <layer number="151" name="HeatSink" color="7" fill="1" visible="no" active="yes"/>
 <layer number="152" name="_bDocu" color="7" fill="1" visible="yes" active="yes"/>
+<layer number="153" name="FabDoc1" color="6" fill="1" visible="no" active="no"/>
+<layer number="154" name="FabDoc2" color="2" fill="1" visible="no" active="no"/>
+<layer number="155" name="FabDoc3" color="7" fill="15" visible="no" active="no"/>
 <layer number="199" name="Contour" color="7" fill="1" visible="yes" active="yes"/>
 <layer number="200" name="200bmp" color="1" fill="10" visible="no" active="yes"/>
@@
 <layer number="223" name="223bmp" color="24" fill="1" visible="no" active="no"/>
 <layer number="224" name="224bmp" color="25" fill="1" visible="no" active="no"/>
+<layer number="231" name="Eagle3D_PG1" color="7" fill="1" visible="no" active="no"/>
+<layer number="232" name="Eagle3D_PG2" color="7" fill="1" visible="no" active="no"/>
+<layer number="233" name="Eagle3D_PG3" color="7" fill="1" visible="no" active="no"/>
 <layer number="248" name="Housing" color="7" fill="1" visible="yes" active="yes"/>
 <layer number="249" name="Edge" color="7" fill="1" visible="yes" active="yes"/>
@@
 <part name="PWR4" library="supply" deviceset="-15V" device=""/>
 <part name="GND2" library="supply" deviceset="GND" device=""/>
-<part name="R2" library="resistors" deviceset="R" device="-0207/10" value="56k"/>
+<part name="R2" library="resistors" deviceset="?" device="56K(TH)" value="56K(TH)"/>
 <part name="DA1" library="ic-ti" deviceset="TL072" device="IP"/>
 <part name="VD1" library="diodes" deviceset="?" device="1N4148"/>
 <part name="VD2" library="diodes" deviceset="?" device="1N4148"/>
-<part name="R3" library="resistors" deviceset="R" device="-0207/10" value="150k"/>
-<part name="R4" library="resistors" deviceset="R" device="-0207/10" value="1.8k"/>
-<part name="C7" library="capacitors-electrolytic" deviceset="C" device="-E1,5-4" value="1u/50V"/>
+<part name="R3" library="resistors" deviceset="?" device="150K(TH)" value="150K(TH)"/>
+<part name="R4" library="resistors" deviceset="?" device="1K8(TH)" value="1K8(TH)"/>
+<part name="C7" library="capacitors-electrolytic" deviceset="?" device="1U/50V" value="1U/50V"/>
 <part name="GND7" library="supply" deviceset="GND" device=""/>
 <part name="GND4" library="supply" deviceset="GND" device=""/>
@@
 <part name="DA2" library="ic-fairchild" deviceset="LM2901" device="N"/>
 <part name="VT1" library="transistors-pnp" deviceset="?" device="BC556"/>
-<part name="R18" library="resistors" deviceset="R" device="-0207/10" value="15k"/>
-<part name="R20" library="resistors" deviceset="R" device="-0207/10" value="180R"/>
-<part name="R19" library="resistors" deviceset="R" device="-0207/10" value="1k"/>
-<part name="C8" library="capacitors" deviceset="C" device="-050-025X075" value="47n"/>
+<part name="R18" library="resistors" deviceset="?" device="15K(TH)" value="15K(TH)"/>
+<part name="R20" library="resistors" deviceset="?" device="180R(TH)" value="180R(TH)"/>
+<part name="R19" library="resistors" deviceset="?" device="1K(TH)" value="1K(TH)"/>
+<part name="C8" library="capacitors" deviceset="?" device="47N(FILM)" value="47N(FILM)"/>
 <part name="PWR6" library="supply" deviceset="+15V" device=""/>
 <part name="PWR7" library="supply" deviceset="-15V" device=""/>
@@
 <part name="HL13" library="optoelectronics" deviceset="?(3MM)" device="RED"/>
 <part name="PWR8" library="supply" deviceset="-15V" device=""/>
-<part name="R16" library="resistors" deviceset="R" device="-0207/10" value="12k"/>
-<part name="R17" library="resistors" deviceset="R" device="-0207/10" value="5.6k"/>
-<part name="R15" library="resistors" deviceset="R" device="-0207/10" value="3.3k"/>
-<part name="R14" library="resistors" deviceset="R" device="-0207/10" value="2.2k"/>
-<part name="R13" library="resistors" deviceset="R" device="-0207/10" value="1.5k"/>
-<part name="R12" library="resistors" deviceset="R" device="-0207/10" value="1.2k"/>
-<part name="R11" library="resistors" deviceset="R" device="-0207/10" value="820R"/>
-<part name="R10" library="resistors" deviceset="R" device="-0207/10" value="560R"/>
-<part name="R9" library="resistors" deviceset="R" device="-0207/10" value="330R"/>
-<part name="R8" library="resistors" deviceset="R" device="-0207/10" value="330R"/>
-<part name="R7" library="resistors" deviceset="R" device="-0207/10" value="220R"/>
-<part name="R6" library="resistors" deviceset="R" device="-0207/10" value="220R"/>
-<part name="R5" library="resistors" deviceset="R" device="-0207/10" value="270R"/>
+<part name="R16" library="resistors" deviceset="?" device="12K(TH)" value="12K(TH)"/>
+<part name="R17" library="resistors" deviceset="?" device="5K6(TH)" value="5K6(TH)"/>
+<part name="R15" library="resistors" deviceset="?" device="3K3(TH)" value="3K3(TH)"/>
+<part name="R14" library="resistors" deviceset="?" device="2K2(TH)" value="2K2(TH)"/>
+<part name="R13" library="resistors" deviceset="?" device="1K5(TH)" value="1K5(TH)"/>
+<part name="R12" library="resistors" deviceset="?" device="1K2(TH)" value="1K2(TH)"/>
+<part name="R11" library="resistors" deviceset="?" device="820R(TH)" value="820R(TH)"/>
+<part name="R10" library="resistors" deviceset="?" device="560R(TH)" value="560R(TH)"/>
+<part name="R9" library="resistors" deviceset="?" device="330R(TH)" value="330R(TH)"/>
+<part name="R8" library="resistors" deviceset="?" device="330R(TH)" value="330R(TH)"/>
+<part name="R7" library="resistors" deviceset="?" device="220R(TH)" value="220R(TH)"/>
+<part name="R6" library="resistors" deviceset="?" device="220R(TH)" value="220R(TH)"/>
+<part name="R5" library="resistors" deviceset="?" device="270R(TH)" value="270R(TH)"/>
 <part name="GND6" library="supply" deviceset="GND" device=""/>
 <part name="PWR5" library="supply" deviceset="+15V" device=""/>
 <part name="GND5" library="supply" deviceset="GND" device=""/>
-<part name="C6" library="capacitors" deviceset="C" device="-050-024X44" value="100n"/>
-<part name="C5" library="capacitors" deviceset="C" device="-050-024X44" value="100n"/>
-<part name="C4" library="capacitors" deviceset="C" device="-050-024X44" value="100n"/>
-<part name="C3" library="capacitors" deviceset="C" device="-050-024X44" value="100n"/>
-<part name="C1" library="capacitors-electrolytic" deviceset="C" device="-E2-5" value="10u/35V"/>
-<part name="C2" library="capacitors-electrolytic" deviceset="C" device="-E2-5" value="10u/35V"/>
+<part name="C6" library="capacitors" deviceset="?" device="100N(TH)" value="100N(TH)"/>
+<part name="C5" library="capacitors" deviceset="?" device="100N(TH)" value="100N(TH)"/>
+<part name="C4" library="capacitors" deviceset="?" device="100N(TH)" value="100N(TH)"/>
+<part name="C3" library="capacitors" deviceset="?" device="100N(TH)" value="100N(TH)"/>
+<part name="C1" library="capacitors-electrolytic" deviceset="?" device="10U/35V" value="10U/35V"/>
+<part name="C2" library="capacitors-electrolytic" deviceset="?" device="10U/35V" value="10U/35V"/>
 <part name="GND1" library="supply" deviceset="GND" device=""/>
 <part name="PWR1" library="supply" deviceset="+15V" device=""/>
 <part name="PWR2" library="supply" deviceset="-15V" device=""/>
+<part name="PCB1" library="module-footprints" deviceset="GENERIC" device="-LOGO" value="R-PREAMP MTR rev.A"/>
 </parts>
 <sheets>
@@
 <instance part="PWR1" gate="G$1" x="25.4" y="106.68" rot="R90"/>
 <instance part="PWR2" gate="G$1" x="25.4" y="86.36" rot="R90"/>
+<instance part="PCB1" gate="G$1" x="48.26" y="152.4"/>
 </instances>
 <busses>
