File: pcb-main.brd (EAGLE design)
At the start: 100 x 80 mm, 91 parts, among them U1 SHHN000A3CL41Z, U2 F15S48

Commit message: Update
Parts:
- removed C21: 10u/50V, capacitors-electrolytic:E2-5
- removed DA1: LM317, regulators-linear:TO220H-HEATSINK
- removed DA2: LM337, regulators-linear:TO220H-HEATSINK
- removed R4: 1k, resistors:R-0207/10
- removed R5, R6: 412R, resistors:R-0207/10
- removed S1, S2: (no value), switches:JP1-SOLDER
- removed VD2, VD3, VD6, VD7: 1N4004GP, diodes:DO41-10
- removed VD4, VD5: LM329, diodes-zener:TO92
- added L2: BL01RN1A1F1J, inductors:BL01RN1A
- added U4: (no value), module-footprints:F-DIP8-HEATSINK
- C1: value 10u/50V -> 10u/35V
- C2: value 100u/25V -> 10u/35V; device capacitors-electrolytic:E2,5-7 -> capacitors-electrolytic:E2-5
- C20: value 100u/25V -> 100u/63V; device capacitors-electrolytic:E2,5-7 -> capacitors-electrolytic:E5-10,5
- C3: value 100u/25V -> 33u/25V; device capacitors-electrolytic:E2,5-7 -> capacitors-electrolytic:E2-5
- C4, C5: value 100n -> 100u/25V; device capacitors:C050-025X075 -> capacitors-electrolytic:E2,5-7
- C6: value 47u/35V -> 100n; device capacitors-electrolytic:E2-5 -> capacitors:C050-024X044
- C7, C9: value 47u/35V -> 100u/25V; device capacitors-electrolytic:E2-5 -> capacitors-electrolytic:E2,5-7
- C8: value 47u/35V -> 100u/63V; device capacitors-electrolytic:E2-5 -> capacitors-electrolytic:E5-10,5
- R1, R2: value 1.5k -> 2.2R
- R11, R12: value 6.81k -> 6.81k*
- R3: value 1k -> 2.2R
- U1: value SHHN000A3CL41Z -> IH1224SH; device regulators-switch-mode:DC/DC-C1 -> regulators-switch-mode:SIP7
- U2: value F15S48 -> RS3-1215D; device regulators-switch-mode:SIP3 -> regulators-switch-mode:SIP8
- moved C20 83.0 mm to (8.50, 47.5), turned to 90 degrees
- moved R7 55.2 mm to (31.0, 36.0)
- moved R3 43.0 mm to (16.5, 61.0), turned to 270 degrees
- moved R1 42.9 mm to (56.0, 74.0), turned to 270 degrees
- moved C6 38.8 mm to (16.5, 54.0), turned to 180 degrees
- moved C19 37.7 mm to (50.0, 20.0), turned to 270 degrees
- moved U1 35.5 mm to (44.0, 77.0)
- moved R15 34.7 mm to (50.0, 27.0), turned to 180 degrees
- moved VD12 31.5 mm to (9.50, 61.0), turned to 90 degrees
- moved R16 28.0 mm to (50.0, 29.5), turned to 180 degrees
- moved C3 26.9 mm to (16.5, 50.0), turned to 0 degrees
- moved C8 26.4 mm to (38.5, 47.5)
- moved C9 25.8 mm to (47.5, 49.0), turned to 180 degrees
- moved C7 25.5 mm to (54.5, 49.0), turned to 180 degrees
- moved R2 21.5 mm to (29.0, 61.0), turned to 270 degrees
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Connections:
- removed net N$20: S1.1, U1.3
- removed net N$3 (its old number): C21.+, L1.1, VD12.C
- new net N$7: R1.1, U1.7
- net +12V: now also C7.+, U4.8; no longer C8.+, DA1.2, R1.2, R3.2, VD2.A, VD7.C
- net +15V: now also C4.+, R2.2, U4.1; no longer C2.+, C4.2, DA1.3, S2.2, U1.4, U2.1, VD2.C
- net +48V: now also C8.+, R1.2; no longer S2.1, U2.3
- net -12V: now also U4.5; no longer DA2.3, R2.1, R4.1, VD3.C, VD6.A
- net -15V: now also C5.-, R3.2, U4.4; no longer C3.-, C5.1, DA2.2, U1.6, VD3.A
- net CHASSIS: now also C2.-, C3.-, C6.1, U2.1; no longer C21.-, S1.2
- net GND: now also C4.-, C5.+, U2.7, U4.2, U4.3, U4.6, U4.7; no longer C2.-, C3.+, C4.1, C5.2, C6.+, R5.2, R6.1, U2.2
- net N$1: now also C2.+, L2.2, U2.2; no longer C7.+, DA1.1, R1.1, VD5.2, VD7.A
- net N$5: now also C3.+, C6.2, L1.1, L2.1, VD12.C; no longer R3.1, R6.2, VD5.3
- net N$8: now also R2.1, U2.6; no longer C6.-, DA2.1, R2.2, VD4.3, VD6.C
- net N$9: now also R3.1, U2.8; no longer R4.2, R5.1, VD4.2

Commit message: Switch footprint fix
Connections:
- removed net N$42: SA1.NO2, XP2.5
- net +15V: no longer SA1.C2
- net N$23: now also SA1.NO1; no longer SA1.NC2
Changed lines of the file:
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@@
 <wire x1="69.81" y1="49.77" x2="69.016" y2="57.5" width="0" layer="19" extent="1-1"/>
 <wire x1="53.23" y1="49" x2="59.5" y2="56.04" width="0" layer="19" extent="1-1"/>
+<wire x1="48.77" y1="49" x2="53.23" y2="49" width="0" layer="19" extent="1-1"/>
 <wire x1="59.5" y1="44.46" x2="53.23" y2="49" width="0" layer="19" extent="1-1"/>
-<wire x1="48.77" y1="49" x2="53.23" y2="49" width="0" layer="19" extent="1-1"/>
 <wire x1="38.5" y1="44.96" x2="48.77" y2="49" width="0" layer="19" extent="1-1"/>
 <wire x1="28.73" y1="51" x2="38.5" y2="44.96" width="0" layer="19" extent="1-1"/>
@@
 <wire x1="90.81" y1="44.81" x2="83" y2="52.54" width="0" layer="19" extent="1-1"/>
 <wire x1="94" y1="43.54" x2="90.81" y2="44.81" width="0" layer="19" extent="1-1"/>
+<wire x1="55.08" y1="29.5" x2="59.5" y2="44.46" width="0" layer="19" extent="1-1"/>
+<wire x1="55.08" y1="27" x2="55.08" y2="29.5" width="0" layer="19" extent="1-1"/>
+<wire x1="8.5" y1="50.04" x2="24.27" y2="51" width="0" layer="19" extent="1-1"/>
 <wire x1="31" y1="30.92" x2="38.5" y2="44.96" width="0" layer="19" extent="1-1"/>
 <wire x1="21.04" y1="28.5" x2="31" y2="30.92" width="0" layer="19" extent="1-1"/>
@@
 <wire x1="35.5" y1="9.46" x2="28.255" y2="6.985" width="0" layer="19" extent="1-1"/>
 <wire x1="35.5" y1="1.46" x2="35.5" y2="9.46" width="0" layer="19" extent="1-1"/>
-<wire x1="8.5" y1="50.04" x2="24.27" y2="51" width="0" layer="19" extent="1-1"/>
-<wire x1="55.08" y1="29.5" x2="59.5" y2="44.46" width="0" layer="19" extent="1-1"/>
-<wire x1="55.08" y1="27" x2="55.08" y2="29.5" width="0" layer="19" extent="1-1"/>
 <wire x1="46.54" y1="77" x2="56.065" y2="62.27" width="0" layer="19" extent="1-1"/>
 <wire x1="81.54" y1="28.5" x2="90.81" y2="44.81" width="0" layer="19" extent="1-1"/>
@@
 <contactref element="VD14" pad="C"/>
 <contactref element="VD1" pad="2"/>
+<contactref element="SA2" pad="NC2"/>
 <contactref element="SA2" pad="NO1"/>
-<contactref element="SA2" pad="NC2"/>
 <wire x1="76.23" y1="18.19" x2="82.81" y2="16" width="0" layer="19" extent="1-1"/>
 <wire x1="67.81" y1="24.54" x2="76.23" y2="18.19" width="0" layer="19" extent="1-1"/>
@@
 <contactref element="R11" pad="2"/>
 <contactref element="R12" pad="2"/>
-<contactref element="SA1" pad="NC2"/>
-<wire x1="31" y1="41.08" x2="69.73" y2="14.24" width="0" layer="19" extent="1-1"/>
+<contactref element="SA1" pad="NO1"/>
+<wire x1="31" y1="41.08" x2="72.27" y2="9.16" width="0" layer="19" extent="1-1"/>
 <wire x1="18" y1="41.08" x2="31" y2="41.08" width="0" layer="19" extent="1-1"/>
 <wire x1="15" y1="41.08" x2="18" y2="41.08" width="0" layer="19" extent="1-1"/>
@@
 </signal>
 <signal name="+15V">
-<contactref element="SA1" pad="C2"/>
 <contactref element="XP2" pad="1"/>
 <contactref element="U4" pad="1"/>
 <contactref element="C4" pad="+"/>
 <contactref element="R2" pad="2"/>
-<wire x1="69.73" y1="11.7" x2="88.73" y2="14.54" width="0" layer="19" extent="1-1"/>
-<wire x1="31.27" y1="51" x2="69.73" y2="11.7" width="0" layer="19" extent="1-1"/>
+<wire x1="31.27" y1="51" x2="88.73" y2="14.54" width="0" layer="19" extent="1-1"/>
 <wire x1="29" y1="55.92" x2="31.27" y2="51" width="0" layer="19" extent="1-1"/>
 <wire x1="31.935" y1="64.81" x2="29" y2="55.92" width="0" layer="19" extent="1-1"/>
@@
 <wire x1="24" y1="76.39" x2="30.5" y2="75.484" width="0" layer="19" extent="1-1"/>
 <wire x1="15.2" y1="69.7" x2="24" y2="76.39" width="0" layer="19" extent="1-1"/>
-<wire x1="17.516" y1="50" x2="15.2" y2="69.7" width="0" layer="19" extent="1-1"/>
-<wire x1="19.04" y1="54" x2="17.516" y2="50" width="0" layer="19" extent="1-1"/>
+<wire x1="19.04" y1="54" x2="15.2" y2="69.7" width="0" layer="19" extent="1-1"/>
+<wire x1="17.516" y1="50" x2="19.04" y2="54" width="0" layer="19" extent="1-1"/>
 </signal>
 <signal name="N$15">
@@
 <wire x1="72.27" y1="11.7" x2="38.5" y2="50.04" width="0" layer="19" extent="1-1"/>
 </signal>
-<signal name="N$42">
-<contactref element="SA1" pad="NO2"/>
-<contactref element="XP2" pad="5"/>
-<wire x1="69.73" y1="9.16" x2="88.73" y2="9.46" width="0" layer="19" extent="1-1"/>
-</signal>
 <signal name="N$31">
 <via x="38" y="20" extent="1-16" drill="3.2"/>
@@
 <contactref element="L1" pad="1"/>
 <contactref element="C6" pad="2"/>
+<wire x1="13.96" y1="54" x2="13" y2="55.92" width="0" layer="19" extent="1-1"/>
 <wire x1="9.5" y1="55.92" x2="13" y2="55.92" width="0" layer="19" extent="1-1"/>
 <wire x1="6" y1="55.92" x2="9.5" y2="55.92" width="0" layer="19" extent="1-1"/>
-<wire x1="15.484" y1="50" x2="13" y2="55.92" width="0" layer="19" extent="1-1"/>
-<wire x1="13.96" y1="54" x2="15.484" y2="50" width="0" layer="19" extent="1-1"/>
+<wire x1="15.484" y1="50" x2="13.96" y2="54" width="0" layer="19" extent="1-1"/>
 </signal>
 <signal name="N$7">

Commit message: Main Board
Parts:
- added PCB1: R-PREAMP rev.A, module-footprints:F-LOGO
- C1, C2: value 10u/35V -> 10U/35V(11MM)
- C10, C35: value 47p -> 47P(TH)
- C11, C12, C19, C33, C34: value 470p -> 470P(FILM)
- C13, C14, C29, C30: value 47u/35V -> 47U/35V(NP)
- C15, C16: value 100p -> 100P(FILM)
- C17, C18: value 47u/63V -> 47U/63V
- C20, C8: value 100u/63V -> 100U/63V
- C22, C23, C25, C26, C41, C42, C6: value 100n -> 100N(TH)
- C24, C43: value 3300u/6.3V -> 3300U/6V3
- C27, C28: value 47u/35V -> 47U/35V
- C3: value 33u/25V -> 47U/35V
- C31, C32: value 330n -> 330N(FILM)
- C36: value 22p -> 22P(TH)
- C4, C5, C7, C9: value 100u/25V -> 100U/25V
- R1, R2, R3: value 2.2R -> 2R2(TH)
- R10, R9: value 4.99k -> 4K99*(TH)
- R11, R12: value 6.81k* -> 6K81*(TH)
- R13, R14: value 47R -> 47R(TH)
- R15, R16: value 1.21k -> 1K21*(TH)
- R18: value 5R -> 5R(TH)
- R19, R8: value 22R -> 20R(TH)
- R20, R22: value 9.1k -> 9K1(TH)
- R23: value 1k -> 1K(TH)
- R7: value 100k -> 100K(TH)
- U1: value IH1224SH -> IH1224DH
- U3: value (none) -> 56DP30-GAIN
- XS4: value PJ-051AH -> 712RA; device connectors:PJ-051AH -> connectors:SWITCHCRAFT-L712RA
- moved C31 19.0 mm to (73.0, 63.0), turned to 90 degrees
- moved C32 19.0 mm to (73.0, 71.0)
- moved XS2 5.00 mm to (85.0, 80.0)
- moved L1 3.00 mm to (6.00, 58.0)
- moved L2 3.00 mm to (13.0, 58.0)
- moved VD12 3.00 mm to (9.50, 58.0)
- moved C20 1.00 mm to (8.50, 46.5)
- moved C7 1.00 mm to (54.5, 48.0)
- moved C8 1.00 mm to (38.5, 46.5)
- moved C9 1.00 mm to (47.5, 48.0)
- moved R1 1.00 mm to (56.0, 73.0)
- moved R2 1.00 mm to (29.0, 62.0)
- moved R3 1.00 mm to (16.5, 62.0)
- moved C3 0.50 mm to (17.0, 50.0)
- moved C6 0.50 mm to (17.0, 54.0)
Connections:
- net CHASSIS: now also XS4.S; no longer XS4.3
- net N$2: now also XS4.P; no longer XS4.1

Commit message: Add component value for LT3032-12 module
Parts:
- U4: value (none) -> F-LT3032-12
Changed lines of the file:
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@@
 <element name="U1" library="regulators-switch-mode" package="SIP7" value="IH1224DH" x="44" y="77"/>
 <element name="U2" library="regulators-switch-mode" package="SIP8" value="RS3-1215D" x="24" y="67.5" rot="R270"/>
-<element name="U4" library="module-footprints" package="F-DIP8-HEATSINK" value="" x="44" y="61" rot="R270"/>
+<element name="U4" library="module-footprints" package="F-DIP8-HEATSINK" value="F-LT3032-12" x="44" y="61" rot="R270"/>
 <element name="L1" library="inductors" package="BL01RN1A" value="BL01RN1A1F1J" x="6" y="58" rot="R90">
 <attribute name="MOUSER" value="81-BL01RN1A1F1J" x="6" y="58" size="1.778" layer="27" rot="R90" display="off"/>

Commit message: Change DC Connector
Parts:
- XS4: value 712RA -> 722RA
Changed lines of the file:
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@@
 <elements>
 <element name="E$1" library="enclosure" package="B*-080" value="" x="0" y="0"/>
-<element name="XS4" library="connectors" package="SWITCHCRAFT-L712RA" value="712RA" x="10" y="80" rot="R270">
+<element name="XS4" library="connectors" package="SWITCHCRAFT-L712RA" value="722RA" x="10" y="80" rot="R270">
 <attribute name="MOUSER" value="502-722RA" x="10" y="80" size="1.778" layer="27" rot="R270" display="off"/>
 </element>

Commit message: PCB Routing
Parts:
- turned C24 to 90 degrees
- turned C30 to 180 degrees
- turned C43 to 90 degrees
- turned R23 to 180 degrees
Routing:
- net -15V: track 0.00 -> 159.2 mm
- net +15V: track 0.00 -> 157.6 mm
- net -12V: track 0.00 -> 150.1 mm
- net +48V: track 0.00 -> 141.2 mm
- net +12V: track 0.00 -> 111.9 mm
- net N$23: track 0.00 -> 106.9 mm
- net CHASSIS: track 0.00 -> 68.1 mm
- net N$21: track 0.00 -> 63.8 mm
- net N$40: track 0.00 -> 58.6 mm
- net N$37: track 0.00 -> 54.9 mm
- net N$13: track 0.00 -> 54.8 mm
- net N$11: track 0.00 -> 50.0 mm
- net N$3: track 0.00 -> 47.0 mm
- net N$29: track 0.00 -> 46.2 mm
- net N$33: track 0.00 -> 45.8 mm
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- added copper zone on layer 1, net GND
- added copper zone on layer 16, net GND

Commit message: Change 20R -> 22R
Parts:
- R19, R8: value 20R(TH) -> 22R(TH)
Changed lines of the file:
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@@
 <element name="C27" library="capacitors-electrolytic" package="E2-5" value="47U/35V" x="68" y="57.5"/>
 <element name="C28" library="capacitors-electrolytic" package="E2-5" value="47U/35V" x="62.5" y="57.5" rot="R180"/>
-<element name="R8" library="resistors" package="R-0207/10" value="20R(TH)" x="59.5" y="37.5" rot="R270"/>
-<element name="R19" library="resistors" package="R-0207/10" value="20R(TH)" x="59.5" y="64.5" rot="R90"/>
+<element name="R8" library="resistors" package="R-0207/10" value="22R(TH)" x="59.5" y="37.5" rot="R270"/>
+<element name="R19" library="resistors" package="R-0207/10" value="22R(TH)" x="59.5" y="64.5" rot="R90"/>
 <element name="C29" library="capacitors-electrolytic" package="E5-10,5" value="47U/35V(NP)" x="90" y="51" rot="R90"/>
 <element name="C30" library="capacitors-electrolytic" package="E5-10,5" value="47U/35V(NP)" x="76" y="51" rot="R180"/>
